Commit message: adding nav stack

File: tb4_mpc_description/urdf/icreate/caster.urdf.xacro (robot description, xacro)
@@ -2,5 +2,5 @@
 <robot xmlns:xacro="http://ros.org/wiki/xacro">
 <xacro:macro name="caster" params="name parent_link *origin">
-  <xacro:include filename="$(find nav2_minimal_tb4_description)/urdf/icreate/common_properties.urdf.xacro"/>
+  <xacro:include filename="$(find tb4_mpc_description)/urdf/icreate/common_properties.urdf.xacro"/>
   <xacro:property name="radius" value="${1*cm2m}" />
   <xacro:property name="mass"   value="0.01"/>

File: tb4_mpc_description/urdf/icreate/create3.urdf.xacro (robot description, xacro)
@@ -1,9 +1,9 @@
 <?xml version="1.0" ?>
 <robot name="create3" xmlns:xacro="http://ros.org/wiki/xacro">
-  <xacro:include filename="$(find nav2_minimal_tb4_description)/urdf/icreate/bumper.urdf.xacro" />
-  <xacro:include filename="$(find nav2_minimal_tb4_description)/urdf/icreate/caster.urdf.xacro" />
-  <xacro:include filename="$(find nav2_minimal_tb4_description)/urdf/icreate/common_properties.urdf.xacro"/>
-  <xacro:include filename="$(find nav2_minimal_tb4_description)/urdf/icreate/sensors/imu.urdf.xacro" />
-  <xacro:include filename="$(find nav2_minimal_tb4_description)/urdf/icreate/wheel.urdf.xacro" />
+  <xacro:include filename="$(find tb4_mpc_description)/urdf/icreate/bumper.urdf.xacro" />
+  <xacro:include filename="$(find tb4_mpc_description)/urdf/icreate/caster.urdf.xacro" />
+  <xacro:include filename="$(find tb4_mpc_description)/urdf/icreate/common_properties.urdf.xacro"/>
+  <xacro:include filename="$(find tb4_mpc_description)/urdf/icreate/sensors/imu.urdf.xacro" />
+  <xacro:include filename="$(find tb4_mpc_description)/urdf/icreate/wheel.urdf.xacro" />
   <!-- Gazebo version -->
   <xacro:arg name="gazebo"                       default="ignition" />

File: tb4_mpc_description/urdf/sensors/camera_bracket.urdf.xacro (robot description, xacro)
@@ -1,5 +1,5 @@
 <?xml version="1.0"?>
 <robot xmlns:xacro="http://ros.org/wiki/xacro">
-<xacro:include filename="$(find nav2_minimal_tb4_description)/urdf/icreate/common_properties.urdf.xacro"/>
+<xacro:include filename="$(find tb4_mpc_description)/urdf/icreate/common_properties.urdf.xacro"/>
 <xacro:macro name="camera_bracket" params="name parent_link:=shell_link *origin">
   <xacro:property name="mass" value="0.033"/>
@@ -14,5 +14,5 @@
     <visual>
       <geometry>
-       <mesh filename="package://nav2_minimal_tb4_description/meshes/camera_bracket.dae" scale="1 1 1" />
+       <mesh filename="package://tb4_mpc_description/meshes/camera_bracket.dae" scale="1 1 1" />
       </geometry>
     </visual>

File: tb4_mpc_description/urdf/sensors/oakd.urdf.xacro (robot description, xacro)
@@ -2,5 +2,5 @@
 <robot xmlns:xacro="http://ros.org/wiki/xacro">
 <xacro:macro name="oakd" params="name:=oakd parent_link *origin model:=pro">
-  <xacro:include filename="$(find nav2_minimal_tb4_description)/urdf/icreate/common_properties.urdf.xacro"/>
+  <xacro:include filename="$(find tb4_mpc_description)/urdf/icreate/common_properties.urdf.xacro"/>
   <xacro:property name="mass"       value="0.061"/>
   <xacro:property name="baseline" value="0.075" />
@@ -22,5 +22,5 @@
     <visual>
       <geometry>
-        <mesh filename="package://nav2_minimal_tb4_description/meshes/${name}_${model}.dae" scale="1 1 1" />
+        <mesh filename="package://tb4_mpc_description/meshes/${name}_${model}.dae" scale="1 1 1" />
       </geometry>
     </visual>

File: tb4_mpc_description/urdf/sensors/rplidar.urdf.xacro (robot description, xacro)
@@ -2,5 +2,5 @@
 <robot xmlns:xacro="http://ros.org/wiki/xacro">
 <xacro:macro name="rplidar" params="name parent_link gazebo *origin">
-  <xacro:include filename="$(find nav2_minimal_tb4_description)/urdf/icreate/common_properties.urdf.xacro"/>
+  <xacro:include filename="$(find tb4_mpc_description)/urdf/icreate/common_properties.urdf.xacro"/>
   <xacro:property name="mass"       value="0.17"/>
   <xacro:property name="length_x"   value="${7.1*cm2m}" />
@@ -18,5 +18,5 @@
     <visual>
       <geometry>
-        <mesh filename="package://nav2_minimal_tb4_description/meshes/rplidar.dae" scale="1 1 1" />
+        <mesh filename="package://tb4_mpc_description/meshes/rplidar.dae" scale="1 1 1" />
       </geometry>
     </visual>

File: tb4_mpc_description/urdf/standard/tower_sensor_plate.urdf.xacro (robot description, xacro)
@@ -1,5 +1,5 @@
 <?xml version="1.0"?>
 <robot xmlns:xacro="http://ros.org/wiki/xacro">
-<xacro:include filename="$(find nav2_minimal_tb4_description)/urdf/icreate/common_properties.urdf.xacro"/>
+<xacro:include filename="$(find tb4_mpc_description)/urdf/icreate/common_properties.urdf.xacro"/>
 <xacro:macro name="tower_sensor_plate" params="name parent_link:=shell_link *origin">
   <xacro:property name="link_name" value="${name}"/>
@@ -14,5 +14,5 @@
     <visual>
       <geometry>
-       <mesh filename="package://nav2_minimal_tb4_description/meshes/tower_sensor_plate.dae" scale="1 1 1" />
+       <mesh filename="package://tb4_mpc_description/meshes/tower_sensor_plate.dae" scale="1 1 1" />
       </geometry>
     </visual>

File: tb4_mpc_description/urdf/standard/tower_standoff.urdf.xacro (robot description, xacro)
@@ -1,5 +1,5 @@
 <?xml version="1.0"?>
 <robot xmlns:xacro="http://ros.org/wiki/xacro">
-<xacro:include filename="$(find nav2_minimal_tb4_description)/urdf/icreate/common_properties.urdf.xacro"/>
+<xacro:include filename="$(find tb4_mpc_description)/urdf/icreate/common_properties.urdf.xacro"/>
 <xacro:macro name="tower_standoff" params="name parent_link:=shell_link *origin">
   <xacro:property name="link_name" value="${name}"/>
@@ -15,5 +15,5 @@
       <origin rpy="0 ${pi/2} 0"/>
       <geometry>
-       <mesh filename="package://nav2_minimal_tb4_description/meshes/tower_standoff.dae" scale="1 1 1" />
+       <mesh filename="package://tb4_mpc_description/meshes/tower_standoff.dae" scale="1 1 1" />
       </geometry>
     </visual>

File: tb4_mpc_description/urdf/standard/turtlebot4.urdf.xacro (robot description, xacro)
@@ -2,11 +2,11 @@
 <robot name="turtlebot4" xmlns:xacro="http://ros.org/wiki/xacro">
   <!-- Base create3 model -->
-  <xacro:include filename="$(find nav2_minimal_tb4_description)/urdf/icreate/create3.urdf.xacro" />
-  <xacro:include filename="$(find nav2_minimal_tb4_description)/urdf/sensors/rplidar.urdf.xacro" />
-  <xacro:include filename="$(find nav2_minimal_tb4_description)/urdf/sensors/oakd.urdf.xacro" />
-  <xacro:include filename="$(find nav2_minimal_tb4_description)/urdf/sensors/camera_bracket.urdf.xacro" />
-  <xacro:include filename="$(find nav2_minimal_tb4_description)/urdf/standard/tower_standoff.urdf.xacro" />
-  <xacro:include filename="$(find nav2_minimal_tb4_description)/urdf/standard/tower_sensor_plate.urdf.xacro" />
-  <xacro:include filename="$(find nav2_minimal_tb4_description)/urdf/standard/weight_block.urdf.xacro" />
+  <xacro:include filename="$(find tb4_mpc_description)/urdf/icreate/create3.urdf.xacro" />
+  <xacro:include filename="$(find tb4_mpc_description)/urdf/sensors/rplidar.urdf.xacro" />
+  <xacro:include filename="$(find tb4_mpc_description)/urdf/sensors/oakd.urdf.xacro" />
+  <xacro:include filename="$(find tb4_mpc_description)/urdf/sensors/camera_bracket.urdf.xacro" />
+  <xacro:include filename="$(find tb4_mpc_description)/urdf/standard/tower_standoff.urdf.xacro" />
+  <xacro:include filename="$(find tb4_mpc_description)/urdf/standard/tower_sensor_plate.urdf.xacro" />
+  <xacro:include filename="$(find tb4_mpc_description)/urdf/standard/weight_block.urdf.xacro" />
   <!-- Mechanical properties -->
   <xacro:property name="shell_z_offset"                value="${3*cm2m}" />
@@ -62,10 +62,10 @@
       <origin xyz="0 0 0" rpy="${pi/2} 0 ${pi/2}"/>
       <geometry>
-        <mesh filename="package://nav2_minimal_tb4_description/meshes/shell.dae" scale="1 1 1" />
+        <mesh filename="package://tb4_mpc_description/meshes/shell.dae" scale="1 1 1" />
       </geometry>
     </visual>
     <collision name="shell_collision">
       <geometry>
-        <mesh filename="package://nav2_minimal_tb4_description/meshes/shell_collision.dae" scale="1 1 1" />
+        <mesh filename="package://tb4_mpc_description/meshes/shell_collision.dae" scale="1 1 1" />
       </geometry>
     </collision>

File: tb4_mpc_description/urdf/standard/weight_block.urdf.xacro (robot description, xacro)
@@ -1,5 +1,5 @@
 <?xml version="1.0"?>
 <robot xmlns:xacro="http://ros.org/wiki/xacro">
-<xacro:include filename="$(find nav2_minimal_tb4_description)/urdf/icreate/common_properties.urdf.xacro"/>
+<xacro:include filename="$(find tb4_mpc_description)/urdf/icreate/common_properties.urdf.xacro"/>
 <xacro:macro name="weight_block" params="name parent_link:=base_link *origin">
   <xacro:property name="link_name" value="${name}"/>
@@ -14,5 +14,5 @@
     <visual>
       <geometry>
-       <mesh filename="package://nav2_minimal_tb4_description/meshes/weight_block.dae" scale="1 1 1" />
+       <mesh filename="package://tb4_mpc_description/meshes/weight_block.dae" scale="1 1 1" />
       </geometry>
     </visual>
