Commit message: testing bringup

File: tb4_mpc_description/urdf/icreate/create3.urdf.xacro (robot description, xacro)
@@ -33,5 +33,5 @@
       <origin xyz="0 0 ${body_z_offset + base_link_z_offset}" rpy="0 0 ${pi/2}"/>
       <geometry>
-        <mesh filename="package://nav2_minimal_tb4_description/meshes/body_visual.dae" />
+        <mesh filename="package://tb4_mpc_description/meshes/body_visual.dae" />
       </geometry>
     </visual>
@@ -53,6 +53,6 @@
       gazebo="$(arg gazebo)"
       namespace="$(arg namespace)"
-      visual_mesh="package://nav2_minimal_tb4_description/meshes/bumper_visual.dae"
-      collision_mesh="package://nav2_minimal_tb4_description/meshes/bumper_collision.dae">
+      visual_mesh="package://tb4_mpc_description/meshes/bumper_visual.dae"
+      collision_mesh="package://tb4_mpc_description/meshes/bumper_collision.dae">
     <origin xyz="0 0 ${bumper_offset_z  + base_link_z_offset}"/>
     <inertial>
